File: PCB/RC_Filter_Dsub/RC_Filter_Dsub.sch (KiCad schematic (older format))
At the start: 28 parts, among them J1 M83513_13-D01CP, U1 BondPad, U10 BondPad, U11 BondPad, U12 BondPad, U13 BondPad, U14 BondPad, U15 BondPad, U16 BondPad, U17 BondPad, U18 BondPad, U19 BondPad, U2 BondPad, U20 BondPad, U21 BondPad, U22 BondPad, U23 BondPad, U24 BondPad, U25 BondPad, U26 BondPad, U27 BondPad, U3 BondPad, U4 BondPad, U5 BondPad, U6 BondPad, U7 BondPad, U8 BondPad, U9 BondPad

Commit message: Great
Parts:
- removed U26, U27: BondPad, RC_Filter_Dsub:BondPad, symbol RC_Filter_Dsub:BondPad
- added TP1: TestPoint, TestPoint:TestPoint_Plated_Hole_D2.0mm, symbol Connector:TestPoint
- added TP2: TestPoint, RC_Filter_Dsub:BondPad, symbol Connector:TestPoint
- added U26: logo, RC_Filter_Dsub:sillyPhotons, symbol RC_Filter_Dsub:logo
Connections:
- net labels added: GND
- wire segments 24 -> 23
Changed lines of the file:
@@
-	-1   0    0    1
-$EndComp
-$Comp
-L RC_Filter_Dsub:BondPad U26
-U 1 1 6161F638
-P 5300 5150
-F 0 "U26" H 5242 4935 50  0000 C CNN
-F 1 "BondPad" H 5242 5026 50  0000 C CNN
-F 2 "RC_Filter_Dsub:BondPad" H 5300 5150 50  0001 C CNN
-F 3 "" H 5300 5150 50  0001 C CNN
-	1    5300 5150
 	-1   0    0    1
 $EndComp
@@
 Wire Wire Line
 	5950 5050 6750 5050
-Wire Wire Line
-	5550 5150 6750 5150
-$Comp
-L RC_Filter_Dsub:BondPad U27
-U 1 1 616213E3
-P 4900 5250
-F 0 "U27" H 4842 5035 50  0000 C CNN
-F 1 "BondPad" H 4842 5126 50  0000 C CNN
-F 2 "RC_Filter_Dsub:BondPad" H 4900 5250 50  0001 C CNN
-F 3 "" H 4900 5250 50  0001 C CNN
-	1    4900 5250
-	-1   0    0    1
-$EndComp
-Wire Wire Line
-	5150 5250 6750 5250
 $Comp
 L RC_Filter_Dsub:BondPad U3
@@
 	-1   0    0    1
 $EndComp
+$Comp
+L RC_Filter_Dsub:logo U26
+U 1 1 615F8282
+P 7750 4950
+F 0 "U26" H 7828 4996 50  0000 L CNN
+F 1 "logo" H 7828 4905 50  0000 L CNN
+F 2 "RC_Filter_Dsub:sillyPhotons" H 7750 4950 50  0001 C CNN
+F 3 "" H 7750 4950 50  0001 C CNN
+	1    7750 4950
+	1    0    0    -1
+$EndComp
+$Comp
+L Connector:TestPoint TP1
+U 1 1 6161406B
+P 2450 5300
+F 0 "TP1" H 2508 5418 50  0000 L CNN
+F 1 "TestPoint" H 2508 5327 50  0000 L CNN
+F 2 "TestPoint:TestPoint_Plated_Hole_D2.0mm" H 2650 5300 50  0001 C CNN
+F 3 "~" H 2650 5300 50  0001 C CNN
+	1    2450 5300
+	1    0    0    -1
+$EndComp
+$Comp
+L power:GND #PWR01
+U 1 1 616144D7
+P 2450 5300
+F 0 "#PWR01" H 2450 5050 50  0001 C CNN
+F 1 "GND" H 2455 5127 50  0000 C CNN
+F 2 "" H 2450 5300 50  0001 C CNN
+F 3 "" H 2450 5300 50  0001 C CNN
+	1    2450 5300
+	1    0    0    -1
+$EndComp
+$Comp
+L Connector:TestPoint TP2
+U 1 1 616158F7
+P 2100 5300
+F 0 "TP2" H 2158 5418 50  0000 L CNN
+F 1 "TestPoint" H 2158 5327 50  0000 L CNN
+F 2 "RC_Filter_Dsub:BondPad" H 2300 5300 50  0001 C CNN
+F 3 "~" H 2300 5300 50  0001 C CNN
+	1    2100 5300
+	1    0    0    -1
+$EndComp
+Wire Wire Line
+	2100 5300 2450 5300
+Connection ~ 2450 5300
 $EndSCHEMATC
