File: PCB/RC_Filter_Dsub/Dsub_Bondpad_1Layer.kicad_pcb (KiCad board)
At the start: 2 copper layers, 30.7 x 13.1 mm, 27 parts, among them J1 M83513_13-D01CP, U11 BondPad, U12 BondPad, U13 BondPad, U14 BondPad, U16 BondPad, U17 BondPad, U18 BondPad, U19 BondPad, U2 BondPad, U21 BondPad, U22 BondPad, U23 BondPad, U24 BondPad, U26 logo, U3 BondPad, U4 BondPad, U6 BondPad, U7 BondPad, U8 BondPad, U9 BondPad

Commit message: Great
Parts:
- added 1: BondPad, RC_Filter_Dsub:BondPad, B.Cu at (175.4, 110.1)
- added 10: BondPad, RC_Filter_Dsub:BondPad, B.Cu at (175.4, 123.1)
- added 15: BondPad, RC_Filter_Dsub:BondPad, B.Cu at (175.4, 112.4)
- added 20: BondPad, RC_Filter_Dsub:BondPad, B.Cu at (175.4, 120.0)
- added 25: BondPad, RC_Filter_Dsub:BondPad, B.Cu at (175.4, 126.9)
- added 5: BondPad, RC_Filter_Dsub:BondPad, B.Cu at (175.4, 117.0)
- added J1: M83513_13-D01CP, RC_Filter_Dsub:M83513&slash_13-D01CP, B.Cu at (187.8, 119.3)
- added U11: BondPad, RC_Filter_Dsub:BondPad, B.Cu at (175.4, 125.3)
- added U12: BondPad, RC_Filter_Dsub:BondPad, B.Cu at (175.4, 127.6)
- added U13: BondPad, RC_Filter_Dsub:BondPad, B.Cu at (175.4, 128.4)
- added U14: BondPad, RC_Filter_Dsub:BondPad, B.Cu at (175.4, 111.6)
- added U16: BondPad, RC_Filter_Dsub:BondPad, B.Cu at (175.4, 113.9)
- added U17: BondPad, RC_Filter_Dsub:BondPad, B.Cu at (175.4, 114.7)
- added U18: BondPad, RC_Filter_Dsub:BondPad, B.Cu at (175.4, 116.2)
- added U19: BondPad, RC_Filter_Dsub:BondPad, B.Cu at (175.4, 118.5)
- added U2: BondPad, RC_Filter_Dsub:BondPad, B.Cu at (175.4, 110.9)
- added U21: BondPad, RC_Filter_Dsub:BondPad, B.Cu at (175.4, 122.3)
- added U22: BondPad, RC_Filter_Dsub:BondPad, B.Cu at (175.4, 123.8)
- added U23: BondPad, RC_Filter_Dsub:BondPad, B.Cu at (175.4, 124.6)
- added U24: BondPad, RC_Filter_Dsub:BondPad, B.Cu at (175.4, 126.1)
- added U26: logo, RC_Filter_Dsub:sillyPhotons, B.Cu at (184.8, 107.6)
- added U3: BondPad, RC_Filter_Dsub:BondPad, B.Cu at (175.4, 113.2)
- added U4: BondPad, RC_Filter_Dsub:BondPad, B.Cu at (175.4, 115.4)
- added U6: BondPad, RC_Filter_Dsub:BondPad, B.Cu at (175.4, 117.7)
- added U7: BondPad, RC_Filter_Dsub:BondPad, B.Cu at (175.4, 119.3)
- added U8: BondPad, RC_Filter_Dsub:BondPad, B.Cu at (175.4, 120.8)
- added U9: BondPad, RC_Filter_Dsub:BondPad, B.Cu at (175.4, 121.5)
- moved U26 32.1 mm to (152.0, 107.6), turned to 270 degrees
- moved 1 28.7 mm to (161.4, 110.1), turned to 270 degrees
- moved U2 27.6 mm to (161.4, 110.9), turned to 270 degrees
- moved U14 26.6 mm to (161.4, 111.6), turned to 270 degrees
- moved 15 25.5 mm to (161.4, 112.4), turned to 270 degrees
- moved U3 24.5 mm to (161.4, 113.2), turned to 270 degrees
- moved U16 23.5 mm to (161.4, 113.9), turned to 270 degrees
- moved U17 22.4 mm to (161.4, 114.7), turned to 270 degrees
- moved U4 21.4 mm to (161.4, 115.4), turned to 270 degrees
- moved U18 20.4 mm to (161.4, 116.2), turned to 270 degrees
- moved 5 19.4 mm to (161.4, 117.0), turned to 270 degrees
- moved J1 18.4 mm to (149.0, 119.3), turned to 90 degrees
- moved U6 18.4 mm to (161.4, 117.7), turned to 270 degrees
- moved U19 17.4 mm to (161.4, 118.5), turned to 270 degrees
- moved U7 16.4 mm to (161.4, 119.3), turned to 270 degrees
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Routing:
- net (no net): track 0.00 -> 178.8 mm, vias 4 -> 8
Other:
- board size 30.7 x 13.1 mm -> 37.8 x 30.7 mm
