File: PCB/MicroD25_Bondpad/MicroD25_Bondpad.kicad_pcb (KiCad board)
At the start: 2 copper layers, 31.5 x 15.7 mm, 53 parts, among them J1 M83513_13-D01CP

Commit message: Great
Other:
- board text added: "Folk Lab 2021 Ray"
- board text removed: "Folk Lab 2021 By Ray with <3"

Commit message: Great
Parts:
- removed B26, B27, B28, B29, B30, B31, B32, B33, B34, B35, B36, B37, B38, B39, B40, B41, B42, B43, B44, B45, B46, B47, B48, B49, B50: BondPad, MicroD25_Bondpad:BondPad_B.Cu
Routing:
- net Net-(B32-Pad1): track 25.4 -> 12.5 mm
- net Net-(B33-Pad1): track 25.2 -> 12.6 mm
- net Net-(B1-Pad1): track 25.2 -> 12.6 mm
- net Net-(B2-Pad1): track 25.0 -> 12.5 mm
- net Net-(B31-Pad1): track 24.9 -> 12.5 mm
- net Net-(B28-Pad1): track 24.8 -> 12.4 mm
- net Net-(B29-Pad1): track 24.6 -> 12.3 mm
- net Net-(B30-Pad1): track 24.6 -> 12.3 mm
- net Net-(B15-Pad1): track 19.2 -> 9.43 mm
- net Net-(B34-Pad1): track 19.2 -> 9.61 mm
- net Net-(B17-Pad1): track 19.2 -> 9.61 mm
- net Net-(B10-Pad1): track 19.1 -> 9.54 mm
- net Net-(B16-Pad1): track 19.0 -> 9.51 mm
- net Net-(B11-Pad1): track 18.9 -> 9.43 mm
- net Net-(B14-Pad1): track 18.6 -> 9.32 mm
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
Commit message: Great
Routing:
- net GND: vias 0 -> 2
- added copper zone on B.Cu, net (none)
- removed copper zone on B.Cu, net GND

Commit message: Great
Parts:
- added B26: BondPad, MicroD25_Bondpad:BondPad, F.Cu at (132.8, 129.2)
- added B27: BondPad, MicroD25_Bondpad:BondPad, F.Cu at (153.2, 129.5)
- added B28: BondPad, MicroD25_Bondpad:BondPad_B.Cu, F.Cu at (132.8, 129.2)
- added B29: BondPad, MicroD25_Bondpad:BondPad_B.Cu, F.Cu at (153.2, 129.5)
- added H3: MountingHole_Pad, MicroD25_Bondpad:ToGND, F.Cu at (128.0, 131.8)
- added H4: MountingHole_Pad, MicroD25_Bondpad:ToGND, F.Cu at (158.0, 131.8)
- H1, H2: footprint MountingHole:MountingHole_2.2mm_M2_DIN965_Pad_TopBottom -> MicroD25_Bondpad:BondableMountHole
- moved J1 35.5 mm to (143.0, 143.3)
- moved B1 35.5 mm to (134.6, 128.4)
- moved B10 35.5 mm to (136.1, 128.4)
- moved B11 35.5 mm to (138.4, 128.4)
- moved B12 35.5 mm to (140.7, 128.4)
- moved B13 35.5 mm to (143.0, 128.4)
- moved B14 35.5 mm to (145.3, 128.4)
- moved B15 35.5 mm to (147.6, 128.4)
- moved B16 35.5 mm to (149.9, 128.4)
- moved B17 35.5 mm to (152.1, 128.4)
- moved B18 35.5 mm to (135.4, 128.4)
- moved B19 35.5 mm to (137.7, 128.4)
- moved B2 35.5 mm to (136.9, 128.4)
- moved B20 35.5 mm to (140.0, 128.4)
- moved B21 35.5 mm to (142.2, 128.4)
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Connections:
- H1 pad 1: GND -> Net-(H1-Pad1)
- H2 pad 1: GND -> Net-(H2-Pad1)
Routing:
- added copper zone on B.Cu, net GND
- removed copper zone on B.Cu, net (none)
Other:
- board size 31.5 x 15.7 mm -> 32 x 15.7 mm
