File: PCB/MicroD25_Bondpad/MicroD25_Bondpad.sch (KiCad schematic (older format))
At the start: 55 parts, among them J1 M83513_13-D01CP, U1 RayLogo, U2 UBCLogo

Commit message: Great
Parts:
- removed B28, B29, B30, B31, B32, B33, B34, B35, B36, B37, B38, B39, B40, B41, B42, B43, B44, B45, B46, B47, B48, B49, B50: BondPad, MicroD25_Bondpad:BondPad_B.Cu, symbol MicroD25_Bondpad:BondPad
- removed U1: RayLogo, MicroD25_Bondpad:sillyPhotons, symbol MicroD25_Bondpad:RayLogo
- removed U2: UBCLogo, MicroD25_Bondpad:ubc, symbol MicroD25_Bondpad:UBCLogo
- B26, B27: footprint MicroD25_Bondpad:BondPad_B.Cu -> MicroD25_Bondpad:BondPad
- H1, H2: footprint MountingHole:MountingHole_2.2mm_M2_DIN965_Pad_TopBottom -> MicroD25_Bondpad:BondableMountHole
Connections:
- net GND: now also B26.1, B27.1; no longer H1.1, H2.1
- net at B1.1, J1.2: no longer B26.1
- net at B2.1, J1.3: no longer B27.1
Other:
- moved on the sheet: H1, H2

Commit message: Great
Parts:
- added B28, B29: BondPad, MicroD25_Bondpad:BondPad_B.Cu, symbol MicroD25_Bondpad:BondPad
- added H3, H4: MountingHole_Pad, MicroD25_Bondpad:ToGND, symbol Mechanical:MountingHole_Pad
Connections:
- net GND: now also B28.1, B29.1, H3.1, H4.1
Changed lines of the file:
@@
 $EndComp
 $Comp
-L power:GND #PWR?
+L power:GND #PWR0101
 U 1 1 6168875C
 P 8700 5200
-F 0 "#PWR?" H 8700 4950 50  0001 C CNN
+F 0 "#PWR0101" H 8700 4950 50  0001 C CNN
 F 1 "GND" H 8705 5027 50  0000 C CNN
 F 2 "" H 8700 5200 50  0001 C CNN
@@
 	8700 5050 8700 5200
 Connection ~ 8700 5200
+$Comp
+L MicroD25_Bondpad:BondPad B28
+U 1 1 6168F51F
+P 8850 5050
+F 0 "B28" H 8950 5100 50  0000 C CNN
+F 1 "BondPad" H 9200 5100 50  0000 C CNN
+F 2 "MicroD25_Bondpad:BondPad_B.Cu" H 8850 5050 50  0001 C CNN
+F 3 "" H 8850 5050 50  0001 C CNN
+	1    8850 5050
+	1    0    0    1
+$EndComp
+$Comp
+L MicroD25_Bondpad:BondPad B29
+U 1 1 61690093
+P 8850 5200
+F 0 "B29" H 8950 5250 50  0000 C CNN
+F 1 "BondPad" H 9200 5250 50  0000 C CNN
+F 2 "MicroD25_Bondpad:BondPad_B.Cu" H 8850 5200 50  0001 C CNN
+F 3 "" H 8850 5200 50  0001 C CNN
+	1    8850 5200
+	1    0    0    1
+$EndComp
+$Comp
+L Mechanical:MountingHole_Pad H4
+U 1 1 6169A17E
+P 9400 4350
+F 0 "H4" H 9500 4399 50  0000 L CNN
+F 1 "MountingHole_Pad" H 9650 4400 50  0000 L CNN
+F 2 "MicroD25_Bondpad:ToGND" H 9400 4350 50  0001 C CNN
+F 3 "~" H 9400 4350 50  0001 C CNN
+	1    9400 4350
+	1    0    0    -1
+$EndComp
+$Comp
+L Mechanical:MountingHole_Pad H3
+U 1 1 6169B343
+P 9000 4350
+F 0 "H3" H 9100 4399 50  0000 L CNN
+F 1 "MountingHole_Pad" H 8200 4400 50  0000 L CNN
+F 2 "MicroD25_Bondpad:ToGND" H 9000 4350 50  0001 C CNN
+F 3 "~" H 9000 4350 50  0001 C CNN
+	1    9000 4350
+	1    0    0    -1
+$EndComp
+$Comp
+L power:GND #PWR?
+U 1 1 6169DD7E
+P 9200 4450
+F 0 "#PWR?" H 9200 4200 50  0001 C CNN
+F 1 "GND" H 9205 4277 50  0000 C CNN
+F 2 "" H 9200 4450 50  0001 C CNN
+F 3 "" H 9200 4450 50  0001 C CNN
+	1    9200 4450
+	1    0    0    -1
+$EndComp
+Wire Wire Line
+	9000 4450 9200 4450
+Connection ~ 9200 4450
+Wire Wire Line
+	9200 4450 9400 4450
 $EndSCHEMATC
